File: pcb/v1-0/Page_1.sch (KiCad schematic (older format))
At the start: 70 parts, among them J1 Conn_01x04, J2 Conn_01x01, J3 Conn_01x01, J4 Conn_01x01, J5 Conn_01x02, J6 Conn_01x04, J7 10118194-0001LF, J8 Conn_02x03_Odd_Even, U1 ATtiny3216-S, U2 SI7211-B-00-IV

Commit message: candidate draft
Parts:
- added C2, C3: 2u2, Capacitor_SMD:C_0805_2012Metric, symbol Device:C
- added J9: Conn_01x01, Connector_PinHeader_2.54mm:PinHeader_1x01_P2.54mm_Vertical, symbol Connector_Generic:Conn_01x01
- S1: footprint SW_DS05-127-2-04BK-SMT-TR -> DS05-127-2-04BK-SMT-TR:SW_DS05-127-2-04BK-SMT-TR
- renumbered FID1 to F2, FID2 to F3
Connections:
- net +5V: now also C2.2, C3.2
- net GND: now also C2.1, C3.1
- net LED_ROW0: now also J9.1 (Pin_1)
Other:
- note added: "Development Test Point"
Changed lines of the file:
@@
 $EndComp
 $Comp
-L Mechanical:Fiducial FID1
+L Mechanical:Fiducial F2
 U 1 1 5F0CEAB1
 P 6200 7450
-F 0 "FID1" H 6285 7496 50  0000 L CNN
+F 0 "F2" H 6285 7496 50  0000 L CNN
 F 1 "Fiducial" H 6285 7405 50  0000 L CNN
 F 2 "Fiducial:Fiducial_1mm_Mask2mm" H 6200 7450 50  0001 C CNN
@@
 $EndComp
 $Comp
-L Mechanical:Fiducial FID2
+L Mechanical:Fiducial F3
 U 1 1 5F0CEAB7
 P 6200 7650
-F 0 "FID2" H 6285 7696 50  0000 L CNN
+F 0 "F3" H 6285 7696 50  0000 L CNN
 F 1 "Fiducial" H 6285 7605 50  0000 L CNN
 F 2 "Fiducial:Fiducial_1mm_Mask2mm" H 6200 7650 50  0001 C CNN
@@
 F 0 "S1" H 10100 6049 50  0000 C CNN
 F 1 "DS05-127-2-04BK-SMT-TR" H 10100 5958 50  0000 C CNN
-F 2 "SW_DS05-127-2-04BK-SMT-TR" H 10100 5500 50  0001 L BNN
+F 2 "DS05-127-2-04BK-SMT-TR:SW_DS05-127-2-04BK-SMT-TR" H 10100 5500 50  0001 L BNN
 F 3 "V0.0" H 10100 5500 50  0001 L BNN
 F 4 "Manufacturer Recommendations" H 10100 5500 50  0001 L BNN "Field4"
@@
 NoConn ~ 3500 7400
 NoConn ~ 3500 7500
+$Comp
+L Connector_Generic:Conn_01x01 J9
+U 1 1 5F7B8020
+P 10000 1000
+F 0 "J9" H 10080 1042 50  0000 L CNN
+F 1 "Conn_01x01" H 10080 951 50  0000 L CNN
+F 2 "Connector_PinHeader_2.54mm:PinHeader_1x01_P2.54mm_Vertical" H 10000 1000 50  0001 C CNN
+F 3 "~" H 10000 1000 50  0001 C CNN
+	1    10000 1000
+	1    0    0    -1
+$EndComp
+Text GLabel 9800 1000 0    50   Input ~ 0
+LED_ROW0
+$Comp
+L Device:C C2
+U 1 1 5F800E02
+P 750 1200
+F 0 "C2" V 498 1200 50  0000 C CNN
+F 1 "2u2" V 589 1200 50  0000 C CNN
+F 2 "Capacitor_SMD:C_0805_2012Metric" H 788 1050 50  0001 C CNN
+F 3 "~" H 750 1200 50  0001 C CNN
+	1    750  1200
+	-1   0    0    1
+$EndComp
+$Comp
+L power:+5V #PWR0218
+U 1 1 5F801A0C
+P 750 1050
+F 0 "#PWR0218" H 750 900 50  0001 C CNN
+F 1 "+5V" H 765 1223 50  0000 C CNN
+F 2 "" H 750 1050 50  0001 C CNN
+F 3 "" H 750 1050 50  0001 C CNN
+	1    750  1050
+	1    0    0    -1
+$EndComp
+$Comp
+L power:GND #PWR0219
+U 1 1 5F801EF6
+P 750 1350
+F 0 "#PWR0219" H 750 1100 50  0001 C CNN
+F 1 "GND" H 755 1177 50  0000 C CNN
+F 2 "" H 750 1350 50  0001 C CNN
+F 3 "" H 750 1350 50  0001 C CNN
+	1    750  1350
+	1    0    0    -1
+$EndComp
+$Comp
+L Device:C C3
+U 1 1 5F8033EB
+P 750 4500
+F 0 "C3" V 498 4500 50  0000 C CNN
+F 1 "2u2" V 589 4500 50  0000 C CNN
+F 2 "Capacitor_SMD:C_0805_2012Metric" H 788 4350 50  0001 C CNN
+F 3 "~" H 750 4500 50  0001 C CNN
+	1    750  4500
+	-1   0    0    1
+$EndComp
+$Comp
+L power:+5V #PWR0220
+U 1 1 5F8033F1
+P 750 4350
+F 0 "#PWR0220" H 750 4200 50  0001 C CNN
+F 1 "+5V" H 765 4523 50  0000 C CNN
+F 2 "" H 750 4350 50  0001 C CNN
+F 3 "" H 750 4350 50  0001 C CNN
+	1    750  4350
+	1    0    0    -1
+$EndComp
+$Comp
+L power:GND #PWR0221
+U 1 1 5F8033F7
+P 750 4650
+F 0 "#PWR0221" H 750 4400 50  0001 C CNN
+F 1 "GND" H 755 4477 50  0000 C CNN
+F 2 "" H 750 4650 50  0001 C CNN
+F 3 "" H 750 4650 50  0001 C CNN
+	1    750  4650
+	1    0    0    -1
+$EndComp
+Text Notes 9550 800  0    50   ~ 0
+Development Test Point
+Wire Notes Line
+	9000 1350 11200 1350
 $EndSCHEMATC
