File: pcb/v1-0/pcb.kicad_pcb (KiCad board)
At the start: 2 copper layers, 254 x 40.6 mm, 30 parts, among them J1 10118194-0001LF, J2 Conn_02x02_Odd_Even, J3 Conn_02x03_Odd_Even, J4 Conn_01x01, J5 Conn_01x04, J6 Conn_01x04, U1 ATtiny3216-S, U2 SI7211-B-00-IV

Commit message: consider program over custom USB and remove 100 mil UPDI header
Parts:
- added D100: WS2812B, WS2812B:LED_WS2812B_PLCC4_5.0x5.0mm_P3.2mm, F.Cu at (147.0, -83.2)
- added D101: WS2812B, WS2812B:LED_WS2812B_PLCC4_5.0x5.0mm_P3.2mm, F.Cu at (130.2, -83.2)
- added D102: WS2812B, WS2812B:LED_WS2812B_PLCC4_5.0x5.0mm_P3.2mm, F.Cu at (163.9, -96.4)
- added D103: WS2812B, WS2812B:LED_WS2812B_PLCC4_5.0x5.0mm_P3.2mm, F.Cu at (172.3, -103.0)
- added D104: WS2812B, WS2812B:LED_WS2812B_PLCC4_5.0x5.0mm_P3.2mm, F.Cu at (180.7, -109.6)
- added D13: WS2812B, WS2812B:LED_WS2812B_PLCC4_5.0x5.0mm_P3.2mm, F.Cu at (274.4, 81.2)
- added D14: WS2812B, WS2812B:LED_WS2812B_PLCC4_5.0x5.0mm_P3.2mm, F.Cu at (264.8, 81.2)
- added D15: WS2812B, WS2812B:LED_WS2812B_PLCC4_5.0x5.0mm_P3.2mm, F.Cu at (255.1, 81.2)
- added D16: WS2812B, WS2812B:LED_WS2812B_PLCC4_5.0x5.0mm_P3.2mm, F.Cu at (245.5, 81.2)
- added D17: WS2812B, WS2812B:LED_WS2812B_PLCC4_5.0x5.0mm_P3.2mm, F.Cu at (235.8, 81.2)
- added D18: WS2812B, WS2812B:LED_WS2812B_PLCC4_5.0x5.0mm_P3.2mm, F.Cu at (226.2, 81.2)
- added D19: WS2812B, WS2812B:LED_WS2812B_PLCC4_5.0x5.0mm_P3.2mm, F.Cu at (216.5, 81.2)
- added D20: WS2812B, WS2812B:LED_WS2812B_PLCC4_5.0x5.0mm_P3.2mm, F.Cu at (206.9, 81.2)
- added D21: WS2812B, WS2812B:LED_WS2812B_PLCC4_5.0x5.0mm_P3.2mm, F.Cu at (197.2, 81.2)
- added D22: WS2812B, WS2812B:LED_WS2812B_PLCC4_5.0x5.0mm_P3.2mm, F.Cu at (187.6, 81.2)
- added D23: WS2812B, WS2812B:LED_WS2812B_PLCC4_5.0x5.0mm_P3.2mm, F.Cu at (177.9, 81.2)
- added D24: WS2812B, WS2812B:LED_WS2812B_PLCC4_5.0x5.0mm_P3.2mm, F.Cu at (168.2, 81.2)
- added D25: WS2812B, WS2812B:LED_WS2812B_PLCC4_5.0x5.0mm_P3.2mm, F.Cu at (158.6, 81.2)
- added D26: WS2812B, WS2812B:LED_WS2812B_PLCC4_5.0x5.0mm_P3.2mm, F.Cu at (166.7, -168.0)
- added D27: WS2812B, WS2812B:LED_WS2812B_PLCC4_5.0x5.0mm_P3.2mm, F.Cu at (152.7, -154.8)
- added D28: WS2812B, WS2812B:LED_WS2812B_PLCC4_5.0x5.0mm_P3.2mm, F.Cu at (205.9, -53.7)
- added D29: WS2812B, WS2812B:LED_WS2812B_PLCC4_5.0x5.0mm_P3.2mm, F.Cu at (143.3, -146.5)
- added D30: WS2812B, WS2812B:LED_WS2812B_PLCC4_5.0x5.0mm_P3.2mm, F.Cu at (130.2, -136.7)
- added D31: WS2812B, WS2812B:LED_WS2812B_PLCC4_5.0x5.0mm_P3.2mm, F.Cu at (121.8, -130.0)
- added D32: WS2812B, WS2812B:LED_WS2812B_PLCC4_5.0x5.0mm_P3.2mm, F.Cu at (152.7, -161.4)
- added D33: WS2812B, WS2812B:LED_WS2812B_PLCC4_5.0x5.0mm_P3.2mm, F.Cu at (165.2, -128.5)
- added D34: WS2812B, WS2812B:LED_WS2812B_PLCC4_5.0x5.0mm_P3.2mm, F.Cu at (147.0, -139.9)
- added D35: WS2812B, WS2812B:LED_WS2812B_PLCC4_5.0x5.0mm_P3.2mm, F.Cu at (186.4, -154.8)
- added D36: WS2812B, WS2812B:LED_WS2812B_PLCC4_5.0x5.0mm_P3.2mm, F.Cu at (138.6, -126.7)
- added D37: WS2812B, WS2812B:LED_WS2812B_PLCC4_5.0x5.0mm_P3.2mm, F.Cu at (155.5, -128.3)
- added D38: WS2812B, WS2812B:LED_WS2812B_PLCC4_5.0x5.0mm_P3.2mm, F.Cu at (176.9, -148.2)
- added D39: WS2812B, WS2812B:LED_WS2812B_PLCC4_5.0x5.0mm_P3.2mm, F.Cu at (186.4, -161.4)
- added D40: WS2812B, WS2812B:LED_WS2812B_PLCC4_5.0x5.0mm_P3.2mm, F.Cu at (163.9, -141.6)
- added D41: WS2812B, WS2812B:LED_WS2812B_PLCC4_5.0x5.0mm_P3.2mm, F.Cu at (177.9, -154.8)
- added D42: WS2812B, WS2812B:LED_WS2812B_PLCC4_5.0x5.0mm_P3.2mm, F.Cu at (169.5, -154.8)
- added D43: WS2812B, WS2812B:LED_WS2812B_PLCC4_5.0x5.0mm_P3.2mm, F.Cu at (155.5, -134.9)
- added D44: WS2812B, WS2812B:LED_WS2812B_PLCC4_5.0x5.0mm_P3.2mm, F.Cu at (147.0, -126.7)
- added D45: WS2812B, WS2812B:LED_WS2812B_PLCC4_5.0x5.0mm_P3.2mm, F.Cu at (168.5, -148.2)
- added D46: WS2812B, WS2812B:LED_WS2812B_PLCC4_5.0x5.0mm_P3.2mm, F.Cu at (155.5, -141.6)
- added D47: WS2812B, WS2812B:LED_WS2812B_PLCC4_5.0x5.0mm_P3.2mm, F.Cu at (177.9, -161.4)
- added D48: WS2812B, WS2812B:LED_WS2812B_PLCC4_5.0x5.0mm_P3.2mm, F.Cu at (183.5, -168.0)
- added D49: WS2812B, WS2812B:LED_WS2812B_PLCC4_5.0x5.0mm_P3.2mm, F.Cu at (147.0, -133.3)
- added D50: WS2812B, WS2812B:LED_WS2812B_PLCC4_5.0x5.0mm_P3.2mm, F.Cu at (138.6, -139.9)
- added D51: WS2812B, WS2812B:LED_WS2812B_PLCC4_5.0x5.0mm_P3.2mm, F.Cu at (155.5, -83.2)
- added D52: WS2812B, WS2812B:LED_WS2812B_PLCC4_5.0x5.0mm_P3.2mm, F.Cu at (147.0, -109.6)
- added D53: WS2812B, WS2812B:LED_WS2812B_PLCC4_5.0x5.0mm_P3.2mm, F.Cu at (138.6, -116.3)
- added D54: WS2812B, WS2812B:LED_WS2812B_PLCC4_5.0x5.0mm_P3.2mm, F.Cu at (130.2, -109.6)
- added D55: WS2812B, WS2812B:LED_WS2812B_PLCC4_5.0x5.0mm_P3.2mm, F.Cu at (121.8, -103.0)
- added D56: WS2812B, WS2812B:LED_WS2812B_PLCC4_5.0x5.0mm_P3.2mm, F.Cu at (113.4, -96.4)
- added D57: WS2812B, WS2812B:LED_WS2812B_PLCC4_5.0x5.0mm_P3.2mm, F.Cu at (130.2, -116.3)
- added D58: WS2812B, WS2812B:LED_WS2812B_PLCC4_5.0x5.0mm_P3.2mm, F.Cu at (121.8, -109.6)
- added D59: WS2812B, WS2812B:LED_WS2812B_PLCC4_5.0x5.0mm_P3.2mm, F.Cu at (113.4, -103.0)
- added D60: WS2812B, WS2812B:LED_WS2812B_PLCC4_5.0x5.0mm_P3.2mm, F.Cu at (163.9, -89.8)
- added D61: WS2812B, WS2812B:LED_WS2812B_PLCC4_5.0x5.0mm_P3.2mm, F.Cu at (113.4, -109.6)
- added D62: WS2812B, WS2812B:LED_WS2812B_PLCC4_5.0x5.0mm_P3.2mm, F.Cu at (147.0, -116.3)
- added D63: WS2812B, WS2812B:LED_WS2812B_PLCC4_5.0x5.0mm_P3.2mm, F.Cu at (172.3, -83.2)
- added D64: WS2812B, WS2812B:LED_WS2812B_PLCC4_5.0x5.0mm_P3.2mm, F.Cu at (180.7, -96.4)
- added D65: WS2812B, WS2812B:LED_WS2812B_PLCC4_5.0x5.0mm_P3.2mm, F.Cu at (172.3, -89.8)
- added D66: WS2812B, WS2812B:LED_WS2812B_PLCC4_5.0x5.0mm_P3.2mm, F.Cu at (217.5, -53.7)
- added D67: WS2812B, WS2812B:LED_WS2812B_PLCC4_5.0x5.0mm_P3.2mm, F.Cu at (163.9, -83.2)
- added D68: WS2812B, WS2812B:LED_WS2812B_PLCC4_5.0x5.0mm_P3.2mm, F.Cu at (180.7, -103.0)
- added D69: WS2812B, WS2812B:LED_WS2812B_PLCC4_5.0x5.0mm_P3.2mm, F.Cu at (172.3, -96.4)
- added D70: WS2812B, WS2812B:LED_WS2812B_PLCC4_5.0x5.0mm_P3.2mm, F.Cu at (121.8, -116.3)
- added D71: WS2812B, WS2812B:LED_WS2812B_PLCC4_5.0x5.0mm_P3.2mm, F.Cu at (163.9, -116.3)
- added D72: WS2812B, WS2812B:LED_WS2812B_PLCC4_5.0x5.0mm_P3.2mm, F.Cu at (155.5, -109.6)
- added D73: WS2812B, WS2812B:LED_WS2812B_PLCC4_5.0x5.0mm_P3.2mm, F.Cu at (147.0, -103.0)
- added D74: WS2812B, WS2812B:LED_WS2812B_PLCC4_5.0x5.0mm_P3.2mm, F.Cu at (138.6, -96.4)
- added D75: WS2812B, WS2812B:LED_WS2812B_PLCC4_5.0x5.0mm_P3.2mm, F.Cu at (130.2, -89.8)
- added D76: WS2812B, WS2812B:LED_WS2812B_PLCC4_5.0x5.0mm_P3.2mm, F.Cu at (121.8, -83.2)
- added D77: WS2812B, WS2812B:LED_WS2812B_PLCC4_5.0x5.0mm_P3.2mm, F.Cu at (155.5, -116.3)
- added D78: WS2812B, WS2812B:LED_WS2812B_PLCC4_5.0x5.0mm_P3.2mm, F.Cu at (113.4, -89.8)
- added D79: WS2812B, WS2812B:LED_WS2812B_PLCC4_5.0x5.0mm_P3.2mm, F.Cu at (138.6, -103.0)
- added D80: WS2812B, WS2812B:LED_WS2812B_PLCC4_5.0x5.0mm_P3.2mm, F.Cu at (225.9, -53.7)
- added D81: WS2812B, WS2812B:LED_WS2812B_PLCC4_5.0x5.0mm_P3.2mm, F.Cu at (130.2, -96.4)
- added D82: WS2812B, WS2812B:LED_WS2812B_PLCC4_5.0x5.0mm_P3.2mm, F.Cu at (121.8, -89.8)
- added D83: WS2812B, WS2812B:LED_WS2812B_PLCC4_5.0x5.0mm_P3.2mm, F.Cu at (113.4, -83.2)
- added D84: WS2812B, WS2812B:LED_WS2812B_PLCC4_5.0x5.0mm_P3.2mm, F.Cu at (113.4, -116.3)
- added D85: WS2812B, WS2812B:LED_WS2812B_PLCC4_5.0x5.0mm_P3.2mm, F.Cu at (138.6, -109.6)
- added D86: WS2812B, WS2812B:LED_WS2812B_PLCC4_5.0x5.0mm_P3.2mm, F.Cu at (130.2, -103.0)
- added D87: WS2812B, WS2812B:LED_WS2812B_PLCC4_5.0x5.0mm_P3.2mm, F.Cu at (121.8, -96.4)
- added D88: WS2812B, WS2812B:LED_WS2812B_PLCC4_5.0x5.0mm_P3.2mm, F.Cu at (155.5, -89.8)
- added D89: WS2812B, WS2812B:LED_WS2812B_PLCC4_5.0x5.0mm_P3.2mm, F.Cu at (138.6, -89.8)
- added D90: WS2812B, WS2812B:LED_WS2812B_PLCC4_5.0x5.0mm_P3.2mm, F.Cu at (147.0, -96.4)
- added D91: WS2812B, WS2812B:LED_WS2812B_PLCC4_5.0x5.0mm_P3.2mm, F.Cu at (155.5, -103.0)
- added D92: WS2812B, WS2812B:LED_WS2812B_PLCC4_5.0x5.0mm_P3.2mm, F.Cu at (163.9, -109.6)
- added D93: WS2812B, WS2812B:LED_WS2812B_PLCC4_5.0x5.0mm_P3.2mm, F.Cu at (172.3, -116.3)
- added D94: WS2812B, WS2812B:LED_WS2812B_PLCC4_5.0x5.0mm_P3.2mm, F.Cu at (138.6, -83.2)
- added D95: WS2812B, WS2812B:LED_WS2812B_PLCC4_5.0x5.0mm_P3.2mm, F.Cu at (147.0, -89.8)
- added D96: WS2812B, WS2812B:LED_WS2812B_PLCC4_5.0x5.0mm_P3.2mm, F.Cu at (155.5, -96.4)
- added D97: WS2812B, WS2812B:LED_WS2812B_PLCC4_5.0x5.0mm_P3.2mm, F.Cu at (163.9, -103.0)
- added D98: WS2812B, WS2812B:LED_WS2812B_PLCC4_5.0x5.0mm_P3.2mm, F.Cu at (172.3, -109.6)
- added D99: WS2812B, WS2812B:LED_WS2812B_PLCC4_5.0x5.0mm_P3.2mm, F.Cu at (180.7, -116.3)
- added J7: 10118194-0001LF, microUSB:AMPHENOL_10118194-0001LF, F.Cu at (27.8, 103.7)
- added J8: Conn_02x03_Odd_Even, Connector_PinHeader_2.54mm:PinHeader_2x03_P2.54mm_Vertical_SMD, F.Cu at (35.2, 112.3)
- J1: value 10118194-0001LF -> Conn_01x04; footprint microUSB:AMPHENOL_10118194-0001LF -> Connector_PinHeader_2.54mm:PinHeader_1x04_P2.54mm_Vertical; moved to B.Cu
- J2: value Conn_02x02_Odd_Even -> Conn_01x01; footprint Connector_PinHeader_2.54mm:PinHeader_2x02_P2.54mm_Vertical -> Connector_PinHeader_2.54mm:PinHeader_1x01_P2.54mm_Vertical
- J3: value Conn_02x03_Odd_Even -> Conn_01x01; footprint Connector_PinHeader_2.54mm:PinHeader_2x03_P2.54mm_Vertical_SMD -> PTC:cap_touch
- J4: footprint PTC:cap_touch -> Connector_PinHeader_2.54mm:PinHeader_1x01_P2.54mm_Vertical; moved to B.Cu
- J5: value Conn_01x04 -> Conn_01x02; footprint Connector_PinHeader_2.54mm:PinHeader_1x04_P2.54mm_Vertical -> Connector_PinHeader_2.54mm:PinHeader_1x02_P2.54mm_Vertical
- R1: value TC33X-2-103E -> 470R; footprint TC33X-2-103E:35WR -> Resistor_SMD:R_0805_2012Metric
- R2: value 470R -> TC33X-2-103E; footprint Resistor_SMD:R_0805_2012Metric -> TC33X-2-103E:35WR
- moved J4 245.4 mm to (277.6, 106.7)
- moved J1 231.2 mm to (257.6, 77.6)
- moved D5 183.4 mm to (81.4, 81.2)
- moved D6 183.4 mm to (91.0, 81.2)
- moved D7 174.0 mm to (100.7, 81.2), turned to 180 degrees
- moved D10 172.5 mm to (129.6, 81.2), turned to 180 degrees
- moved D11 170.8 mm to (139.3, 81.2), turned to 180 degrees
- moved D8 165.4 mm to (110.3, 81.2)
- moved D12 161.6 mm to (148.9, 81.2), turned to 180 degrees
- moved D9 157.4 mm to (120.0, 81.2), turned to 180 degrees
- moved D4 42.1 mm to (71.7, 81.2), turned to 180 degrees
- moved J3 34.1 mm to (33.9, 78.1), turned to 0 degrees
- moved J5 28.4 mm to (277.6, 97.8), turned to 0 degrees
- moved D3 28.1 mm to (62.1, 81.2)
- moved R2 18.2 mm to (34.8, 103.9)
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Connections:
- D11 pad 4: Net-(D11-Pad4) -> Net-(D10-Pad2)
- D12 pad 4: Net-(D12-Pad4) -> Net-(D11-Pad2)
- D2 pad 4: LED_ROW1 -> Net-(D1-Pad2)
- D3 pad 4: LED_ROW2 -> Net-(D2-Pad2)
- D4 pad 4: LED_ROW3 -> Net-(D3-Pad2)
- D5 pad 4: Net-(D1-Pad2) -> Net-(D4-Pad2)
- D7 pad 2: Net-(D11-Pad4) -> Net-(D7-Pad2)
- D7 pad 4: Net-(D2-Pad2) -> Net-(D6-Pad2)
- D8 pad 2: Net-(D12-Pad4) -> Net-(D8-Pad2)
- D8 pad 4: Net-(D3-Pad2) -> Net-(D7-Pad2)
- D9 pad 4: Net-(D4-Pad2) -> Net-(D8-Pad2)
- J1 pad 2: Net-(J1-Pad2) -> GND
- J1 pad 3: Net-(J1-Pad3) -> RxD
- J1 pad 4: Net-(J1-Pad4) -> TxD
- J3 pad 1: UPDI_DATA -> PTC
- J4 pad 1: PTC -> TxD
- J5 pad 1: +5V -> GND
- J5 pad 2: GND -> +5V
- R1 pad 1: +5V -> LED_ROW0
- R1 pad 2: BRIGHTNESS -> Net-(R1-Pad2)
- R2 pad 1: LED_ROW0 -> +5V
- R2 pad 2: Net-(R2-Pad2) -> BRIGHTNESS
- U1 pad 5: Net-(R2-Pad2) -> Net-(R1-Pad2)

Commit message: compontnets placedr
Parts:
- removed D102, D103, D104: WS2812B, WS2812B:LED_WS2812B_PLCC4_5.0x5.0mm_P3.2mm
- removed the D64 at (180.7, -96.4)
- removed the D72 at (155.5, -109.6)
- removed the D79 at (138.6, -103.0)
- removed the D91 at (155.5, -103.0)
- removed the D95 at (147.0, -89.8)
- added D100: WS2812B, WS2812B:LED_WS2812B_PLCC4_5.0x5.0mm_P3.2mm, F.Cu at (148.9, 111.9)
- added D71: WS2812B, WS2812B:LED_WS2812B_PLCC4_5.0x5.0mm_P3.2mm, F.Cu at (197.2, 101.6)
- added D92: WS2812B, WS2812B:LED_WS2812B_PLCC4_5.0x5.0mm_P3.2mm, F.Cu at (71.7, 111.9)
- added D93: WS2812B, WS2812B:LED_WS2812B_PLCC4_5.0x5.0mm_P3.2mm, F.Cu at (81.4, 111.9)
- added S1: DS05-127-2-04BK-SMT-TR, DS05-127-2-04BK-SMT-TR:SW_DS05-127-2-04BK-SMT-TR, F.Cu at (35.7, 103.3)
- moved D39 290.7 mm to (42.8, 91.4)
- moved D26 280.9 mm to (274.4, 91.4)
- moved D41 272.1 mm to (62.1, 91.4)
- moved D27 270.5 mm to (264.8, 91.4)
- moved D48 265.0 mm to (129.6, 91.4)
- moved D42 264.9 mm to (71.7, 91.4)
- moved D32 260.8 mm to (216.5, 91.4)
- moved D47 259.4 mm to (120.0, 91.4)
- moved D29 259.0 mm to (245.5, 91.4)
- moved D40 258.2 mm to (52.4, 91.4)
- moved D76 258.1 mm to (274.4, 111.9)
- moved D90 257.7 mm to (52.4, 111.9)
- moved D77 253.0 mm to (264.8, 111.9)
- moved D89 252.5 mm to (42.8, 111.9)
- moved D30 251.3 mm to (235.8, 91.4)
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- renumbered D65 to D64, D66 to D65, D67 to D66, D68 to D67, D69 to D68, D70 to D69, D71 to D70, D73 to D72, D74 to D73, D75 to D74, D76 to D75, D78 to D76, D80 to D78, D81 to D79, D82 to D80, D83 to D81, D84 to D82, D85 to D83, D86 to D84, D87 to D85, D88 to D86, D89 to D87, D90 to D88, D92 to D89, D93 to D90, D94 to D91, D97 to D94, D98 to D95, D100 to D97, D101 to D98, FID1 to F1, FID2 to FID1, FID3 to FID2
Connections:
- D60 pad 1: +5V -> Net-(D60-Pad1)
- D63 pad 4: Net-(D62-Pad2) -> Net-(D63-Pad4)
- D64 pad 2: Net-(D64-Pad4) (its old number) -> Net-(D63-Pad4)
- D75 pad 4: Net-(D76-Pad4) -> Net-(D62-Pad2)
- D76 pad 2: Net-(D78-Pad2) (its old number) -> Net-(D76-Pad2)
- D76 pad 4: Net-(D64-Pad2) -> Net-(D63-Pad2)
- D77 pad 2: Net-(D76-Pad4) -> Net-(D77-Pad2)
- D77 pad 4: Net-(D63-Pad2) -> Net-(D76-Pad2)
- D78 pad 4: Net-(D79-Pad2) (its old number) -> Net-(D77-Pad2)
- D94 pad 2: Net-(D96-Pad4) -> Net-(D93-Pad4)
- D95 pad 4: Net-(D98-Pad4) -> Net-(D95-Pad4)
- D97 pad 2: Net-(D100-Pad2) -> Net-(D96-Pad4)
- D98 pad 4: Net-(D101-Pad4) -> Net-(D98-Pad4)
- J7 pad 4: Net-(J7-Pad4) -> USB_UPDI
- JP2 pad 1: Net-(D64-Pad4) (its old number) -> Net-(D63-Pad4)
- JP2 pad 2: Net-(D78-Pad2) (its old number) -> Net-(D76-Pad2)
- U1 pad 2: Net-(U1-Pad2) -> SW1
- U1 pad 3: Net-(U1-Pad3) -> SW2
- U1 pad 4: Net-(U1-Pad4) -> SW3

Commit message: pre-zone fill
Parts:
- moved JP1 5.08 mm to (269.6, 91.4)
- moved JP2 5.08 mm to (269.6, 111.8)
Connections:
- J7 pad S2: Net-(J7-PadS1) -> Net-(J7-PadS2)
- J7 pad S3: Net-(J7-PadS1) -> Net-(J7-PadS3)
- J7 pad S4: Net-(J7-PadS1) -> Net-(J7-PadS4)
- J7 pad S5: Net-(J7-PadS1) -> Net-(J7-PadS5)
- J7 pad S6: Net-(J7-PadS1) -> Net-(J7-PadS6)
- U1 pad 2: SW1 -> SW3
- U1 pad 4: SW3 -> SW1
Routing:
- net TxD: track 0.00 -> 290.4 mm, vias 0 -> 2
- net RxD: track 0.00 -> 284.2 mm, vias 0 -> 1
- net GND: track 0.00 -> 65.5 mm
- net UPDI_DATA: track 0.00 -> 42.3 mm, vias 0 -> 2
- net BRIGHTNESS: track 0.00 -> 22.7 mm, vias 0 -> 2
- net Net-(D13-Pad4): track 0.00 -> 22.7 mm, vias 0 -> 1
- net Net-(D63-Pad4): track 0.00 -> 14.5 mm, vias 0 -> 1
- net SW1: track 0.00 -> 14.0 mm
- net USB_UPDI: track 0.00 -> 13.8 mm
- net SW2: track 0.00 -> 13.2 mm
- net SW3: track 0.00 -> 12.5 mm
- net LED_CONT: track 0.00 -> 11.9 mm
- net Net-(D63-Pad2): track 0.00 -> 11.5 mm
- net Net-(D13-Pad2): track 0.00 -> 11.5 mm
- net Net-(D76-Pad2): track 0.00 -> 8.97 mm, vias 0 -> 1
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
Commit message: candidate draft
Routing:
- net +5V: track 5.37 -> 58.4 mm, vias 0 -> 174
- net GND: track 65.5 -> 103.0 mm, vias 0 -> 255
- net TxD: track 290.4 -> 291.4 mm
- added copper zone on B.Cu, net +5V
- added copper zone on F.Cu, net +5V
- added copper zone on B.Cu, net GND
- added copper zone on F.Cu, net GND

Commit message: candidate draft
Parts:
- added C2: 2u2, Capacitor_SMD:C_0805_2012Metric, F.Cu at (153.8, 81.1)
- added C3: 2u2, Capacitor_SMD:C_0805_2012Metric, F.Cu at (153.8, 91.4)
- added C4: 2u2, Capacitor_SMD:C_0805_2012Metric, F.Cu at (153.8, 101.8)
- added C5: 2u2, Capacitor_SMD:C_0805_2012Metric, F.Cu at (153.8, 111.9)
- added J9: Conn_01x01, Connector_PinHeader_2.54mm:PinHeader_1x01_P2.54mm_Vertical, F.Cu at (47.6, 86.7)
- renumbered FID1 to F2, FID2 to F3
Routing:
- net GND: track 103.0 -> 113.6 mm
- net +5V: track 58.4 -> 69.0 mm, vias 174 -> 171
- net LED_ROW0: track 3.00 -> 12.4 mm
Other:
- board text added: "+5V"
- board text added: "+5V GND > TxD < RxD"
- board text added: "+5V GND RxD > TxD <"
- board text added: "2"
- board text added: "6"
- board text added: "GND"
- board text added: "Github: Name Plate Scott Almond v1.0"
- board text added: "J3: Touch sensor"
- board text added: "J8: UPDI 1: UPDI Data 2: +5V 6: GND"
- board text added: "ON"
- board text added: "R2: Brightness adjust"
- board text added: "RxD >"
- board text added: "S1: Configuration settings"
- board text added: "TxD <"
- board text added: "U2: Magnetic sensor"
